File: ISCAS25_Blinker/ISCAS25_Blinker.kicad_pcb (KiCad board)
At the start: 2 copper layers, 85 x 66.9 mm, 26 parts, among them J1 USB_C_Receptacle_PowerOnly_6P, Q1 BC846, Q2 BC857, U2 NE555D

Commit message: Finished but not panelized
Parts:
- removed LOGO, LOGO2: LOGO, LOGO
- added ? (x5): , Graphics, F.Cu at (106.5, 98.8)
- added ?: , DrillHole, F.Cu at (176.5, 143.5)
- added ? (x5): , Graphics, F.Cu at (190.5, 152.8)
- added ?: , DrillHole, F.Cu at (157.5, 143.5)
- added ?: , Graphics, B.Cu at (106.5, 98.8)
- added ?: , Graphics, B.Cu at (190.5, 152.8)
- added ?: , DrillHole, F.Cu at (119.4, 143.5)
- added ?: , DrillHole, F.Cu at (138.5, 143.5)
- added C2: 0.1uF, Capacitor_SMD:C_0603_1608Metric, B.Cu at (176.2, 81.9)
- added G***: LOGO, LOGO, F.Cu at (176.4, 81.6)
- added G***: LOGO, LOGO, F.Cu at (147.5, 85.6)
- added QR: QR, LOGO, F.Cu at (120.6, 80.4)
- added S1: SLW-1277545-3A-RA-N-D, Library:SW_SLW-1277545-3A-RA-N-D, B.Cu at (108.4, 80.0)
- added mouse-bite-2.54mm-4.66mm: VAL**, mouse-bite:mouse-bite-2.54mm-4.66mm, F.Cu at (259.6, 93.5)
- added mouse-bite-2.54mm-4.66mm: VAL**, mouse-bite:mouse-bite-2.54mm-4.66mm, F.Cu at (209.4, 93.5)
- added mouse-bite-2.54mm-4.66mm: VAL**, mouse-bite:mouse-bite-2.54mm-4.66mm, F.Cu at (199.6, 93.5)
- added mouse-bite-2.54mm-4.66mm: VAL**, mouse-bite:mouse-bite-2.54mm-4.66mm, F.Cu at (269.4, 93.5)
- C1: footprint Capacitor_THT:C_Rect_L11.0mm_W6.4mm_P10.00mm_MKT -> Capacitor_THT:CP_Radial_D6.3mm_P2.50mm
- moved J1 114.5 mm to (149.0, 102.6)
- moved R4 66.1 mm to (179.3, 59.6)
- moved R5 65.5 mm to (175.2, 59.6)
- moved R6 62.6 mm to (165.2, 59.6)
- moved R7 62.1 mm to (161.1, 59.6)
- moved R9 59.8 mm to (124.1, 59.6)
- moved R2 59.6 mm to (144.3, 59.6)
- moved R8 59.5 mm to (128.2, 59.6)
- moved R1 59.3 mm to (148.4, 59.6)
- moved R3 46.8 mm to (174.7, 77.6), turned to 180 degrees
- moved Q1 38.3 mm to (163.3, 76.6), turned to 90 degrees
- moved U2 37.1 mm to (181.5, 78.2)
- moved ? 33.9 mm to (105.8, 27.1) (x3)
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Connections:
- J1 pad A9: +5V -> Net-(J1-VBUS-PadA9)
- J1 pad B9: +5V -> Net-(J1-VBUS-PadA9)
Routing:
- net +5V: track 0.00 -> 223.7 mm, vias 0 -> 7
- net /LED_1_Driver: track 0.00 -> 201.2 mm, vias 0 -> 2
- net /LED_2_Driver: track 0.00 -> 122.2 mm, vias 0 -> 6
- net GND: track 0.00 -> 64.9 mm, vias 0 -> 15
- net Net-(J1-VBUS-PadA9): track 0.00 -> 60.7 mm
- net Net-(Q1-B): track 0.00 -> 47.8 mm
- net Net-(D1-A-Pad3): track 0.00 -> 22.1 mm
- net Net-(D3-A-Pad3): track 0.00 -> 19.9 mm
- net Net-(D1-A-Pad4): track 0.00 -> 17.5 mm
- net Net-(D2-A-Pad3): track 0.00 -> 17.2 mm
- net Net-(D3-A-Pad4): track 0.00 -> 15.4 mm
- net Net-(D2-A-Pad4): track 0.00 -> 13.1 mm
- net Net-(D4-A-Pad3): track 0.00 -> 11.5 mm
- net Net-(D4-A-Pad4): track 0.00 -> 7.70 mm
- net Net-(U2-Q): track 0.00 -> 3.53 mm
- added copper zone on B.Cu, net GND
- added copper zone on F.Cu, net GND
- added copper zone on B.Cu, net Net-(J1-VBUS-PadA9)
Other:
- board size 85 x 66.9 mm -> 86.1 x 125.7 mm
- board text added: "Designed by Juan M. Montes, ATC, Universidad de Sevilla"
- board text added: "ISCAS25_Blinker v1.0"
- board text added: "Visit my ORCID profile 0000-0002-0983-2386"
- board text added: "github.com/juamonsan/ISCAS25_PCB"

Commit message: Final assembly
Parts:
- removed mouse-bite-2.54mm-4.66mm (x4): VAL**, mouse-bite:mouse-bite-2.54mm-4.66mm
- added ? (x5): , Graphics, F.Cu at (95.4, 29.0)
- added ?: , Graphics, B.Cu at (95.4, 29.0)
- added mouse-bite-3mm-6mm: VAL**, mouse-bite:mouse-bite-3mm-6mm, F.Cu at (109.2, 97.2)
- added mouse-bite-3mm-6mm: VAL**, mouse-bite:mouse-bite-3mm-6mm, F.Cu at (117.2, 135.1)
- added mouse-bite-3mm-6mm: VAL**, mouse-bite:mouse-bite-3mm-6mm, F.Cu at (158.9, 135.1)
- added mouse-bite-3mm-6mm: VAL**, mouse-bite:mouse-bite-3mm-6mm, F.Cu at (166.1, 97.2)
- moved ? 11.1 mm to (95.4, 98.7) (x6)
- moved J1 11.1 mm to (137.9, 102.6)
- moved D3 10.6 mm to (147.4, 45.6)
- moved Q2 10.6 mm to (158.1, 78.5)
- moved ? 10.6 mm to (95.4, 29.0) (x6)
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Routing:
- net +5V: track 223.7 -> 228.2 mm
- net GND: track 64.9 -> 63.3 mm
- net /LED_2_Driver: track 122.2 -> 123.8 mm
- net Net-(J1-VBUS-PadA9): track 60.7 -> 61.6 mm
Other:
- board size 86.1 x 125.7 mm -> 85 x 123.8 mm
